File: hardware/rx.sch (EAGLE design)
At the start: 48 parts, among them IC1 TL072P, IC2 MEGA8-P, IC3 TL072P, Q1 20MHz

Commit message: ...
Parts:
- removed C13: 22pF, rcl:C-EU025-025X050
- removed C14, C15: 100nF, rcl:C-EU025-025X050
- removed C9: 10uF, rcl:CPOL-EUE2.5-6
- removed D1: 3.6V, diode:ZENER-DIODEZD-2.5
- removed IC2: MEGA8-P, atmel:MEGA8-P
- removed ISP1: AVRISP-6, adafruit:AVRISP-6
- removed L2: 10uH, rcl:L-EU0204/5
- removed Q1: 20MHz, crystal:CRYSTALHC49S
- removed X1: (no value), con-berg:PN87520
- added C3: 100nF, rcl:C-EU025-025X050
- added C4: 1nF, rcl:C-EU025-025X050
- added JP1: OUT, pinhead:PINHD-1X1
- added JP3: GND, pinhead:PINHD-1X1
- added JP4: SUPPLY, pinhead:PINHD-1X3
- added JP5: BAT, pinhead:PINHD-1X2
- added JP6: SW-1, pinhead:PINHD-1X1
- added JP7: SW-2, pinhead:PINHD-1X1
- added R7: 4.7k, rcl:R-EU_0204/7
- added R8: B, rcl:R-EU_0204/5
- added T1: BC547, transistor-neu-to92:-NPN-TO92-CBE
- added U$2: BS170-LINE, transistor-small-signal:BS170-LINE
- C1, C18: device rcl:C-EU025-025X050 -> rcl:C-EU075-032X103
- C5: value 22pF -> 1nF
- C6: value 47uF -> 10uF
- C8: value 100nF -> 10uF; device rcl:C-EU025-025X050 -> rcl:CPOL-EUE2.5-6
- D2: value 3.6V -> 1N4148; device diode:ZENER-DIODEZD-2.5 -> diode:DIODE-D-2.5
- IC1, IC3: value TL072P -> LM358N; device linear:TL072P -> linear:LM358N
- R1, R19, R2: device rcl:R-EU_0204/2V -> rcl:R-EU_0207/10
- R10: value 10k -> 1k
- R11: value 2.2k -> A; device rcl:R-EU_0204/2V -> rcl:R-EU_0204/5
- R12: value 68 -> 560; device rcl:R-EU_0204/2V -> rcl:R-EU_0204/7
- R13: value 68 -> 10
- R15, R16: device rcl:R-EU_0204/2V -> rcl:R-EU_0204/5
- R17, R22: value 1k -> 10k; device rcl:R-EU_0204/2V -> rcl:R-EU_0204/5
- R18: value 10k -> 100k
- R20: device rcl:R-EU_0204/2V -> rcl:R-EU_0204/7
- R3: value 1k -> 10k; device rcl:R-EU_0204/2V -> rcl:R-EU_0207/10
- R5: value 100 -> 4.7k; device rcl:R-EU_0204/2V -> rcl:R-EU_0204/7
- R9: value 10k -> 1k; device rcl:R-EU_0204/2V -> rcl:R-EU_0204/5
Connections:
- removed net +5V: C12.1, C8.1, C9.+, IC1P.V+, IC2.VCC@1, ISP1.VCC, L1.2, L2.2, R14.1, R9.2
- removed net N$19: C14.2, IC2.AVCC, L2.1
- removed net N$21: IC2.PB3(MOSI/OC2), ISP1.MOSI
- removed net N$22: IC2.PB4(MISO), ISP1.MISO
- removed net N$23: IC2.PB5(SCK), ISP1.SCK
- new net VCC: C12.1, C3.1, C8.+, IC1P.V+, IC3P.V+, JP7.1, R9.2
- net AGND: now also C5.2, R6.E
- net GND: now also C3.2, C8.-, IC3P.V-, JP3.1, JP4.1, R8.1, T1.E; no longer C13.2, C14.1, C15.2, C5.2, C8.2, C9.-, D1.A, D2.A, IC2.GND, IC2.GND@1, ISP1.GND, X1.4
- net N$10: now also C4.1, R5.2, R7.1; no longer IC2.PD2(INT0), R13.1
- net N$11: now also JP4.2; no longer R11.1, X1.1
- net N$12: now also JP4.3, JP5.2, R12.1, R8.2; no longer D1.C, R13.2, X1.3
- net N$13: now also T1.B; no longer D2.C, R11.2, X1.2
- net N$14: now also D2.A, JP5.1, U$2.S; no longer IC2.PD3(INT1), R12.1
- net N$15: now also R11.1, U$2.D; no longer C13.1, IC2.PB6(XTAL1/TOSC1), Q1.1
- net N$16: now also R13.1, U$2.G; no longer C5.1, IC2.PB7(XTAL2/TOSC2), Q1.2
- net N$17: now also R13.2, T1.C; no longer IC2.PC6(/RESET), ISP1.RST
- net N$18: now also D2.C, JP6.1, L1.2, R11.2, R14.1; no longer C15.1, IC2.AREF
- net N$5: now also R6.S; no longer R6.E
- net N$6: now also C5.1, R7.2; no longer R5.2
- net N$8: now also C4.2, JP1.1; no longer IC2.PC0(ADC0), R6.S
Other:
- note added: "9V NiMH"
- note added: "A = 12V / I_max"
- note added: "B = 0.6V/I_trickle"
- moved on the sheet: C10, C11, C12, C17, C5, C6, C7, IC1B, L1, R10, R11, R12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
